Commit message: More ur sim stuff

File: ur_description/urdf/ur_ignition_plugins.xacro (robot description, xacro)
@@ -1,4 +1,13 @@
 <?xml version="1.0"?>
 <robot xmlns:xacro="http://www.ros.org/wiki/xacro" name="ur_ignition_plugins">
+  <!-- Joint Controller Gains -->
+  <xacro:property name="default_initial_position" value="0"/>
+  <xacro:property name="default_position_p_gain" value="3000"/>
+  <xacro:property name="default_position_d_gain" value="0"/>
+  <xacro:property name="default_position_i_gain" value="100"/>
+  <xacro:property name="default_position_i_min" value="-50"/>
+  <xacro:property name="default_position_i_max" value="50"/>
+  <xacro:property name="default_position_cmd_min" value="-100"/>
+  <xacro:property name="default_position_cmd_max" value="100"/>
   <gazebo>
     <!-- Joint States -->
@@ -8,57 +17,57 @@
       <topic>joint_trajectory</topic>
       <joint_name>shoulder_pan_joint</joint_name>
-      <initial_position>0</initial_position>
-      <position_p_gain>3000</position_p_gain>
-      <position_d_gain>15</position_d_gain>
-      <position_i_gain>1650</position_i_gain>
-      <position_i_min>-15</position_i_min>
-      <position_i_max>15</position_i_max>
-      <position_cmd_min>-87</position_cmd_min>
-      <position_cmd_max>87</position_cmd_max>
+      <initial_position>${default_initial_position}</initial_position>
+      <position_p_gain>${default_position_p_gain}</position_p_gain>
+      <position_d_gain>${default_position_d_gain}</position_d_gain>
+      <position_i_gain>${default_position_i_gain}</position_i_gain>
+      <position_i_min>${default_position_i_min}</position_i_min>
+      <position_i_max>${default_position_i_max}</position_i_max>
+      <position_cmd_min>${default_position_cmd_min}</position_cmd_min>
+      <position_cmd_max>${default_position_cmd_max}</position_cmd_max>
       <joint_name>shoulder_lift_joint</joint_name>
-      <initial_position>0</initial_position>
-      <position_p_gain>3000</position_p_gain>
-      <position_d_gain>15</position_d_gain>
-      <position_i_gain>1650</position_i_gain>
-      <position_i_min>-15</position_i_min>
-      <position_i_max>15</position_i_max>
-      <position_cmd_min>-87</position_cmd_min>
-      <position_cmd_max>87</position_cmd_max>
+      <initial_position>${default_initial_position}</initial_position>
+      <position_p_gain>${default_position_p_gain}</position_p_gain>
+      <position_d_gain>${default_position_d_gain}</position_d_gain>
+      <position_i_gain>${default_position_i_gain}</position_i_gain>
+      <position_i_min>${default_position_i_min}</position_i_min>
+      <position_i_max>${default_position_i_max}</position_i_max>
+      <position_cmd_min>${default_position_cmd_min}</position_cmd_min>
+      <position_cmd_max>${default_position_cmd_max}</position_cmd_max>
       <joint_name>elbow_joint</joint_name>
-      <initial_position>0</initial_position>
-      <position_p_gain>3000</position_p_gain>
-      <position_d_gain>15</position_d_gain>
-      <position_i_gain>1650</position_i_gain>
-      <position_i_min>-15</position_i_min>
-      <position_i_max>15</position_i_max>
-      <position_cmd_min>-87</position_cmd_min>
-      <position_cmd_max>87</position_cmd_max>
+      <initial_position>${default_initial_position}</initial_position>
+      <position_p_gain>${default_position_p_gain}</position_p_gain>
+      <position_d_gain>${default_position_d_gain}</position_d_gain>
+      <position_i_gain>${default_position_i_gain}</position_i_gain>
+      <position_i_min>${default_position_i_min}</position_i_min>
+      <position_i_max>${default_position_i_max}</position_i_max>
+      <position_cmd_min>${default_position_cmd_min}</position_cmd_min>
+      <position_cmd_max>${default_position_cmd_max}</position_cmd_max>
       <joint_name>wrist_1_joint</joint_name>
-      <initial_position>0</initial_position>
-      <position_p_gain>3000</position_p_gain>
-      <position_d_gain>15</position_d_gain>
-      <position_i_gain>1650</position_i_gain>
-      <position_i_min>-15</position_i_min>
-      <position_i_max>15</position_i_max>
-      <position_cmd_min>-87</position_cmd_min>
-      <position_cmd_max>87</position_cmd_max>
+      <initial_position>${default_initial_position}</initial_position>
+      <position_p_gain>${default_position_p_gain}</position_p_gain>
+      <position_d_gain>${default_position_d_gain}</position_d_gain>
+      <position_i_gain>${default_position_i_gain}</position_i_gain>
+      <position_i_min>${default_position_i_min}</position_i_min>
+      <position_i_max>${default_position_i_max}</position_i_max>
+      <position_cmd_min>${default_position_cmd_min}</position_cmd_min>
+      <position_cmd_max>${default_position_cmd_max}</position_cmd_max>
       <joint_name>wrist_2_joint</joint_name>
-      <initial_position>0</initial_position>
-      <position_p_gain>3000</position_p_gain>
-      <position_d_gain>15</position_d_gain>
-      <position_i_gain>1650</position_i_gain>
-      <position_i_min>-15</position_i_min>
-      <position_i_max>15</position_i_max>
-      <position_cmd_min>-87</position_cmd_min>
-      <position_cmd_max>87</position_cmd_max>
+      <initial_position>${default_initial_position}</initial_position>
+      <position_p_gain>${default_position_p_gain}</position_p_gain>
+      <position_d_gain>${default_position_d_gain}</position_d_gain>
+      <position_i_gain>${default_position_i_gain}</position_i_gain>
+      <position_i_min>${default_position_i_min}</position_i_min>
+      <position_i_max>${default_position_i_max}</position_i_max>
+      <position_cmd_min>${default_position_cmd_min}</position_cmd_min>
+      <position_cmd_max>${default_position_cmd_max}</position_cmd_max>
       <joint_name>wrist_3_joint</joint_name>
-      <initial_position>0</initial_position>
-      <position_p_gain>3000</position_p_gain>
-      <position_d_gain>15</position_d_gain>
-      <position_i_gain>1650</position_i_gain>
-      <position_i_min>-15</position_i_min>
-      <position_i_max>15</position_i_max>
-      <position_cmd_min>-87</position_cmd_min>
-      <position_cmd_max>87</position_cmd_max>
+      <initial_position>${default_initial_position}</initial_position>
+      <position_p_gain>${default_position_p_gain}</position_p_gain>
+      <position_d_gain>${default_position_d_gain}</position_d_gain>
+      <position_i_gain>${default_position_i_gain}</position_i_gain>
+      <position_i_min>${default_position_i_min}</position_i_min>
+      <position_i_max>${default_position_i_max}</position_i_max>
+      <position_cmd_min>${default_position_cmd_min}</position_cmd_min>
+      <position_cmd_max>${default_position_cmd_max}</position_cmd_max>
     </plugin>
   </gazebo>

File: ur_description/urdf/ur_macro.xacro (robot description, xacro)
@@ -125,5 +125,5 @@
         </geometry>
       </collision>
-      <xacro:cylinder_inertial radius="${shoulder_inertia_radius}" length="${shoulder_inertia_length}" mass="${shoulder_mass}">
+      <xacro:cylinder_inertial radius="${shoulder_inertia_radius}" length="${shoulder_inertia_length}" mass="1">
         <origin xyz="0 0 0" rpy="0 0 0" />
       </xacro:cylinder_inertial>
@@ -145,5 +145,5 @@
         </geometry>
       </collision>
-      <xacro:cylinder_inertial radius="${upperarm_inertia_radius}" length="${upperarm_inertia_length}" mass="${upper_arm_mass}">
+      <xacro:cylinder_inertial radius="${upperarm_inertia_radius}" length="${upperarm_inertia_length}" mass="1">
         <origin xyz="${-0.5 * upperarm_inertia_length} 0.0 ${upper_arm_inertia_offset}" rpy="0 ${pi/2} 0" />
       </xacro:cylinder_inertial>
@@ -165,5 +165,5 @@
         </geometry>
       </collision>
-      <xacro:cylinder_inertial radius="${forearm_inertia_radius}" length="${forearm_inertia_length}"  mass="${forearm_mass}">
+      <xacro:cylinder_inertial radius="${forearm_inertia_radius}" length="${forearm_inertia_length}"  mass="1">
         <origin xyz="${-0.5 * forearm_inertia_length} 0.0 ${elbow_offset}" rpy="0 ${pi/2} 0" />
       </xacro:cylinder_inertial>
@@ -185,5 +185,5 @@
         </geometry>
       </collision>
-      <xacro:cylinder_inertial radius="${wrist_1_inertia_radius}" length="${wrist_1_inertia_length}"  mass="${wrist_1_mass}">
+      <xacro:cylinder_inertial radius="${wrist_1_inertia_radius}" length="${wrist_1_inertia_length}"  mass="1">
         <origin xyz="0 0 0" rpy="0 0 0" />
       </xacro:cylinder_inertial>
@@ -205,5 +205,5 @@
         </geometry>
       </collision>
-      <xacro:cylinder_inertial radius="${wrist_2_inertia_radius}" length="${wrist_2_inertia_length}"  mass="${wrist_2_mass}">
+      <xacro:cylinder_inertial radius="${wrist_2_inertia_radius}" length="${wrist_2_inertia_length}"  mass="1">
         <origin xyz="0 0 0" rpy="0 0 0" />
       </xacro:cylinder_inertial>
@@ -225,5 +225,5 @@
         </geometry>
       </collision>
-      <xacro:cylinder_inertial radius="${wrist_3_inertia_radius}" length="${wrist_3_inertia_length}"  mass="${wrist_3_mass}">
+      <xacro:cylinder_inertial radius="${wrist_3_inertia_radius}" length="${wrist_3_inertia_length}"  mass="1">
         <origin xyz="0.0 0.0 ${-0.5 * wrist_3_inertia_length}" rpy="0 0 0" />
       </xacro:cylinder_inertial>

Commit message: Better tuning

File: ur_description/urdf/ur_ignition_plugins.xacro (robot description, xacro)
@@ -4,10 +4,10 @@
   <xacro:property name="default_initial_position" value="0"/>
   <xacro:property name="default_position_p_gain" value="3000"/>
-  <xacro:property name="default_position_d_gain" value="0"/>
-  <xacro:property name="default_position_i_gain" value="100"/>
-  <xacro:property name="default_position_i_min" value="-50"/>
-  <xacro:property name="default_position_i_max" value="50"/>
-  <xacro:property name="default_position_cmd_min" value="-100"/>
-  <xacro:property name="default_position_cmd_max" value="100"/>
+  <xacro:property name="default_position_d_gain" value="15"/>
+  <xacro:property name="default_position_i_gain" value="1650"/>
+  <xacro:property name="default_position_i_min" value="-15"/>
+  <xacro:property name="default_position_i_max" value="15"/>
+  <xacro:property name="default_position_cmd_min" value="-87"/>
+  <xacro:property name="default_position_cmd_max" value="87"/>
   <gazebo>
     <!-- Joint States -->

File: ur_description/urdf/ur_macro.xacro (robot description, xacro)
@@ -88,4 +88,6 @@
     <!-- Placeholder for ros2_control transmission which don't yet exist -->
     <!-- links -  main serial chain -->
+    <!-- World link for static base -->
+    <link name="world" />
     <link name="${prefix}base_link"/>
     <link name="${prefix}base_link_inertia">
@@ -102,5 +104,5 @@
         </geometry>
       </collision>
-      <xacro:cylinder_inertial radius="${base_inertia_radius}" length="${base_inertia_length}" mass="1000">
+      <xacro:cylinder_inertial radius="${base_inertia_radius}" length="${base_inertia_length}" mass="${base_mass}">
         <origin xyz="0 0 0" rpy="0 0 0" />
       </xacro:cylinder_inertial>
@@ -119,5 +121,5 @@
         </geometry>
       </collision>
-      <xacro:cylinder_inertial radius="${shoulder_inertia_radius}" length="${shoulder_inertia_length}" mass="1">
+      <xacro:cylinder_inertial radius="${shoulder_inertia_radius}" length="${shoulder_inertia_length}" mass="${shoulder_mass}">
         <origin xyz="0 0 0" rpy="0 0 0" />
       </xacro:cylinder_inertial>
@@ -136,5 +138,5 @@
         </geometry>
       </collision>
-      <xacro:cylinder_inertial radius="${upperarm_inertia_radius}" length="${upperarm_inertia_length}" mass="1">
+      <xacro:cylinder_inertial radius="${upperarm_inertia_radius}" length="${upperarm_inertia_length}" mass="${upper_arm_mass}">
         <origin xyz="${-0.5 * upperarm_inertia_length} 0.0 ${upper_arm_inertia_offset}" rpy="0 ${pi/2} 0" />
       </xacro:cylinder_inertial>
@@ -153,5 +155,5 @@
         </geometry>
       </collision>
-      <xacro:cylinder_inertial radius="${forearm_inertia_radius}" length="${forearm_inertia_length}"  mass="1">
+      <xacro:cylinder_inertial radius="${forearm_inertia_radius}" length="${forearm_inertia_length}"  mass="${forearm_mass}">
         <origin xyz="${-0.5 * forearm_inertia_length} 0.0 ${elbow_offset}" rpy="0 ${pi/2} 0" />
       </xacro:cylinder_inertial>
@@ -170,5 +172,5 @@
         </geometry>
       </collision>
-      <xacro:cylinder_inertial radius="${wrist_1_inertia_radius}" length="${wrist_1_inertia_length}"  mass="1">
+      <xacro:cylinder_inertial radius="${wrist_1_inertia_radius}" length="${wrist_1_inertia_length}"  mass="${wrist_1_mass}">
         <origin xyz="0 0 0" rpy="0 0 0" />
       </xacro:cylinder_inertial>
@@ -187,5 +189,5 @@
         </geometry>
       </collision>
-      <xacro:cylinder_inertial radius="${wrist_2_inertia_radius}" length="${wrist_2_inertia_length}"  mass="1">
+      <xacro:cylinder_inertial radius="${wrist_2_inertia_radius}" length="${wrist_2_inertia_length}"  mass="${wrist_2_mass}">
         <origin xyz="0 0 0" rpy="0 0 0" />
       </xacro:cylinder_inertial>
@@ -204,9 +206,14 @@
         </geometry>
       </collision>
-      <xacro:cylinder_inertial radius="${wrist_3_inertia_radius}" length="${wrist_3_inertia_length}"  mass="1">
+      <xacro:cylinder_inertial radius="${wrist_3_inertia_radius}" length="${wrist_3_inertia_length}"  mass="${wrist_3_mass}">
         <origin xyz="0.0 0.0 ${-0.5 * wrist_3_inertia_length}" rpy="0 0 0" />
       </xacro:cylinder_inertial>
     </link>
     <!-- joints - main serial chain -->
+    <joint name="${prefix}world_joint"  type="fixed">
+      <origin xyz="0 0 0" rpy="0 0 0" />
+      <parent link="world"/>
+      <child link="${prefix}base_link"/>
+    </joint>
     <joint name="${prefix}base_link-base_link_inertia" type="fixed">
       <parent link="${prefix}base_link" />
