Commit message: Add ft_sensor frame.

File: ur_description/urdf/ur_macro.xacro (robot description, xacro)
@@ -312,4 +312,10 @@
       <dynamics damping="0" friction="0"/>
     </joint>
+    <link name="${prefix}ft_frame"/>
+    <joint name="${prefix}wrist_3_link-ft_frame" type="fixed">
+      <parent link="${prefix}wrist_3_link"/>
+      <child link="${prefix}ft_frame"/>
+      <origin xyz="0 0 0" rpy="${pi} 0 0"/>
+    </joint>
     <!-- ROS-Industrial 'base' frame - base_link to UR 'Base' Coordinates transform -->
     <link name="${prefix}base"/>
@@ -334,8 +340,8 @@
     <link name="${prefix}tool0"/>
     <joint name="${prefix}flange-tool0" type="fixed">
+      <parent link="${prefix}flange"/>
+      <child link="${prefix}tool0"/>
       <!-- default toolframe - X+ left, Y+ up, Z+ front -->
       <origin xyz="0 0 0" rpy="${pi/2.0} 0 ${pi/2.0}"/>
-      <parent link="${prefix}flange"/>
-      <child link="${prefix}tool0"/>
     </joint>
   </xacro:macro>

Commit message: Remove visual colors, so colors are read from dae

File: ur_description/urdf/ur_macro.xacro (robot description, xacro)
@@ -95,7 +95,4 @@
           <mesh filename="${base_visual_mesh}"/>
         </geometry>
-        <material name="${base_visual_material_name}">
-          <color rgba="${base_visual_material_color}"/>
-        </material>
       </visual>
       <collision>
@@ -115,7 +112,4 @@
           <mesh filename="${shoulder_visual_mesh}"/>
         </geometry>
-        <material name="${shoulder_visual_material_name}">
-          <color rgba="${shoulder_visual_material_color}"/>
-        </material>
       </visual>
       <collision>
@@ -135,7 +129,4 @@
           <mesh filename="${upper_arm_visual_mesh}"/>
         </geometry>
-        <material name="${upper_arm_visual_material_name}">
-          <color rgba="${upper_arm_visual_material_color}"/>
-        </material>
       </visual>
       <collision>
@@ -155,7 +146,4 @@
           <mesh filename="${forearm_visual_mesh}"/>
         </geometry>
-        <material name="${forearm_visual_material_name}">
-          <color rgba="${forearm_visual_material_color}"/>
-        </material>
       </visual>
       <collision>
@@ -175,7 +163,4 @@
           <mesh filename="${wrist_1_visual_mesh}"/>
         </geometry>
-        <material name="${wrist_1_visual_material_name}">
-          <color rgba="${wrist_1_visual_material_color}"/>
-        </material>
       </visual>
       <collision>
@@ -195,7 +180,4 @@
           <mesh filename="${wrist_2_visual_mesh}"/>
         </geometry>
-        <material name="${wrist_2_visual_material_name}">
-          <color rgba="${wrist_2_visual_material_color}"/>
-        </material>
       </visual>
       <collision>
@@ -215,7 +197,4 @@
           <mesh filename="${wrist_3_visual_mesh}"/>
         </geometry>
-        <material name="${wrist_3_visual_material_name}">
-          <color rgba="${wrist_3_visual_material_color}"/>
-        </material>
       </visual>
       <collision>

Commit message: More organizational changes

File: ur_description/urdf/ur_macro.xacro (robot description, xacro)
@@ -89,6 +89,4 @@
     <!-- Placeholder for ros2_control transmission which don't yet exist -->
     <!-- links -  main serial chain -->
-    <!-- World link for static base -->
-    <link name="world" />
     <link name="${prefix}base_link"/>
     <link name="${prefix}base_link_inertia">
@@ -212,9 +210,4 @@
     </link>
     <!-- joints - main serial chain -->
-    <joint name="${prefix}world_joint"  type="fixed">
-      <origin xyz="0 0 0" rpy="0 0 0" />
-      <parent link="world"/>
-      <child link="${prefix}base_link"/>
-    </joint>
     <joint name="${prefix}base_link-base_link_inertia" type="fixed">
       <parent link="${prefix}base_link" />
@@ -326,8 +319,16 @@
       <child link="${prefix}tool0"/>
     </joint>
-  <!-- Ignition Plugins -->
-  <xacro:if value="${ignition}">
-    <xacro:include filename="ur_ignition_plugins.xacro" />
-  </xacro:if>
+    <!-- Ignition Gazebo -->
+    <xacro:if value="${ignition}">
+      <!-- Create a world link, and a fixed between world and base_link -->
+      <link name="world" />
+      <joint name="${prefix}world_joint"  type="fixed">
+        <origin xyz="0 0 0" rpy="0 0 0" />
+        <parent link="world"/>
+        <child link="${prefix}base_link"/>
+      </joint>
+      <!-- Include Ignition Gazebo Plugins -->
+      <xacro:include filename="ur_ignition_plugins.xacro" />
+    </xacro:if>
   </xacro:macro>
 </robot>

Commit message: Move world link outside xacro if

File: ur_description/urdf/ur_macro.xacro (robot description, xacro)
@@ -319,13 +319,13 @@
       <child link="${prefix}tool0"/>
     </joint>
+    <!-- Create a world link, and a fixed joint between world and base_link -->
+    <link name="world" />
+    <joint name="${prefix}world_joint"  type="fixed">
+      <origin xyz="0 0 0" rpy="0 0 0" />
+      <parent link="world"/>
+      <child link="${prefix}base_link"/>
+    </joint>
     <!-- Ignition Gazebo -->
     <xacro:if value="${ignition}">
-      <!-- Create a world link, and a fixed between world and base_link -->
-      <link name="world" />
-      <joint name="${prefix}world_joint"  type="fixed">
-        <origin xyz="0 0 0" rpy="0 0 0" />
-        <parent link="world"/>
-        <child link="${prefix}base_link"/>
-      </joint>
       <!-- Include Ignition Gazebo Plugins -->
       <xacro:include filename="ur_ignition_plugins.xacro" />

Commit message: added get_mesh macro, updated gazebo simuation launch file, removed ur5 urdf files

File: ur_description/urdf/ur_macro.xacro (robot description, xacro)
@@ -96,5 +96,5 @@
         <origin xyz="0 0 0" rpy="0 0 ${pi}"/>
         <geometry>
-          <mesh filename="file://$(find ${base_visual_mesh['package']})/${base_visual_mesh['path']}"/>
+          <xacro:get_mesh name="base" type="visual"/>
         </geometry>
         <material name="${base_visual_material_name}">
@@ -105,5 +105,5 @@
         <origin xyz="0 0 0" rpy="0 0 ${pi}"/>
         <geometry>
-          <mesh filename="file://$(find ${base_collision_mesh['package']})/${base_collision_mesh['path']}"/>
+          <xacro:get_mesh name="base" type="collision"/>
         </geometry>
       </collision>
@@ -116,5 +116,5 @@
         <origin xyz="0 0 0" rpy="0 0 ${pi}"/>
         <geometry>
-          <mesh filename="file://$(find ${shoulder_visual_mesh['package']})/${shoulder_visual_mesh['path']}"/>
+          <xacro:get_mesh name="shoulder" type="visual"/>
         </geometry>
         <material name="${shoulder_visual_material_name}">
@@ -125,5 +125,5 @@
         <origin xyz="0 0 0" rpy="0 0 ${pi}"/>
         <geometry>
-          <mesh filename="file://$(find ${shoulder_collision_mesh['package']})/${shoulder_collision_mesh['path']}"/>
+          <xacro:get_mesh name="shoulder" type="collision"/>
         </geometry>
       </collision>
@@ -136,5 +136,5 @@
         <origin xyz="0 0 ${shoulder_offset}" rpy="${pi/2} 0 ${-pi/2}"/>
         <geometry>
-          <mesh filename="file://$(find ${upper_arm_visual_mesh['package']})/${upper_arm_visual_mesh['path']}"/>
+          <xacro:get_mesh name="upper_arm" type="visual"/>
         </geometry>
         <material name="${upper_arm_visual_material_name}">
@@ -145,5 +145,5 @@
         <origin xyz="0 0 ${shoulder_offset}" rpy="${pi/2} 0 ${-pi/2}"/>
         <geometry>
-          <mesh filename="file://$(find ${upper_arm_collision_mesh['package']})/${upper_arm_collision_mesh['path']}"/>
+          <xacro:get_mesh name="upper_arm" type="collision"/>
         </geometry>
       </collision>
@@ -156,5 +156,5 @@
         <origin xyz="0 0 ${elbow_offset}" rpy="${pi/2} 0 ${-pi/2}"/>
         <geometry>
-          <mesh filename="file://$(find ${forearm_visual_mesh['package']})/${forearm_visual_mesh['path']}"/>
+          <xacro:get_mesh name="forearm" type="visual"/>
         </geometry>
         <material name="${forearm_visual_material_name}">
@@ -165,5 +165,5 @@
         <origin xyz="0 0 ${elbow_offset}" rpy="${pi/2} 0 ${-pi/2}"/>
         <geometry>
-          <mesh filename="file://$(find ${forearm_collision_mesh['package']})/${forearm_collision_mesh['path']}"/>
+          <xacro:get_mesh name="forearm" type="collision"/>
         </geometry>
       </collision>
@@ -176,5 +176,5 @@
         <origin xyz="0 0 ${wrist_1_visual_offset}" rpy="${pi/2} 0 0"/>
         <geometry>
-          <mesh filename="file://$(find ${wrist_1_visual_mesh['package']})/${wrist_1_visual_mesh['path']}"/>
+          <xacro:get_mesh name="wrist_1" type="visual"/>
         </geometry>
         <material name="${wrist_1_visual_material_name}">
@@ -185,5 +185,5 @@
         <origin xyz="0 0 ${wrist_1_visual_offset}" rpy="${pi/2} 0 0"/>
         <geometry>
-          <mesh filename="file://$(find ${wrist_1_collision_mesh['package']})/${wrist_1_collision_mesh['path']}"/>
+          <xacro:get_mesh name="wrist_1" type="collision"/>
         </geometry>
       </collision>
@@ -196,5 +196,5 @@
         <origin xyz="0 0 ${wrist_2_visual_offset}" rpy="0 0 0"/>
         <geometry>
-          <mesh filename="file://$(find ${wrist_2_visual_mesh['package']})/${wrist_2_visual_mesh['path']}"/>
+          <xacro:get_mesh name="wrist_2" type="visual"/>
         </geometry>
         <material name="${wrist_2_visual_material_name}">
@@ -205,5 +205,5 @@
         <origin xyz="0 0 ${wrist_2_visual_offset}" rpy="0 0 0"/>
         <geometry>
-          <mesh filename="file://$(find ${wrist_2_collision_mesh['package']})/${wrist_2_collision_mesh['path']}"/>
+          <xacro:get_mesh name="wrist_2" type="collision"/>
         </geometry>
       </collision>
@@ -216,5 +216,5 @@
         <origin xyz="0 0 ${wrist_3_visual_offset}" rpy="${pi/2} 0 0"/>
         <geometry>
-          <mesh filename="file://$(find ${wrist_3_visual_mesh['package']})/${wrist_3_visual_mesh['path']}"/>
+          <xacro:get_mesh name="wrist_3" type="visual"/>
         </geometry>
         <material name="${wrist_3_visual_material_name}">
@@ -225,5 +225,5 @@
         <origin xyz="0 0 ${wrist_3_visual_offset}" rpy="${pi/2} 0 0"/>
         <geometry>
-          <mesh filename="file://$(find ${wrist_3_collision_mesh['package']})/${wrist_3_collision_mesh['path']}"/>
+          <xacro:get_mesh name="wrist_3" type="collision"/>
         </geometry>
       </collision>
