Commit message: Make ur and ignition happy

File: ur_description/urdf/ur.urdf.xacro (robot description, xacro)
@@ -38,3 +38,5 @@
      headless_mode="$(arg headless_mode)"
      initial_positions="${load_yaml(initial_positions_file)}" />
+  <!-- Ignition -->
+  <xacro:include filename="ur_ignition_plugins.xacro" />
 </robot>

File: ur_description/urdf/ur_macro.xacro (robot description, xacro)
@@ -105,5 +105,5 @@
         </geometry>
       </collision>
-      <xacro:cylinder_inertial radius="${base_inertia_radius}" length="${base_inertia_length}" mass="${base_mass}">
+      <xacro:cylinder_inertial radius="${base_inertia_radius}" length="${base_inertia_length}" mass="1000">
         <origin xyz="0 0 0" rpy="0 0 0" />
       </xacro:cylinder_inertial>
@@ -250,5 +250,5 @@
          <safety_controller soft_lower_limit="${shoulder_pan_lower_limit + safety_pos_margin}" soft_upper_limit="${shoulder_pan_upper_limit - safety_pos_margin}" k_position="${safety_k_position}" k_velocity="0.0"/>
       </xacro:if>
-      <dynamics damping="0" friction="0"/>
+      <dynamics damping="5" friction="5"/>
     </joint>
     <joint name="${prefix}shoulder_lift_joint" type="revolute">
@@ -262,5 +262,5 @@
          <safety_controller soft_lower_limit="${shoulder_lift_lower_limit + safety_pos_margin}" soft_upper_limit="${shoulder_lift_upper_limit - safety_pos_margin}" k_position="${safety_k_position}" k_velocity="0.0"/>
       </xacro:if>
-      <dynamics damping="0" friction="0"/>
+      <dynamics damping="5" friction="5"/>
     </joint>
     <joint name="${prefix}elbow_joint" type="revolute">
@@ -274,5 +274,5 @@
          <safety_controller soft_lower_limit="${elbow_joint_lower_limit + safety_pos_margin}" soft_upper_limit="${elbow_joint_upper_limit - safety_pos_margin}" k_position="${safety_k_position}" k_velocity="0.0"/>
       </xacro:if>
-      <dynamics damping="0" friction="0"/>
+      <dynamics damping="5" friction="5"/>
     </joint>
     <joint name="${prefix}wrist_1_joint" type="revolute">
@@ -286,5 +286,5 @@
          <safety_controller soft_lower_limit="${wrist_1_lower_limit + safety_pos_margin}" soft_upper_limit="${wrist_1_upper_limit - safety_pos_margin}" k_position="${safety_k_position}" k_velocity="0.0"/>
       </xacro:if>
-      <dynamics damping="0" friction="0"/>
+      <dynamics damping="5" friction="5"/>
     </joint>
     <joint name="${prefix}wrist_2_joint" type="revolute">
@@ -298,5 +298,5 @@
          <safety_controller soft_lower_limit="${wrist_2_lower_limit + safety_pos_margin}" soft_upper_limit="${wrist_2_upper_limit - safety_pos_margin}" k_position="${safety_k_position}" k_velocity="0.0"/>
       </xacro:if>
-      <dynamics damping="0" friction="0"/>
+      <dynamics damping="5" friction="5"/>
     </joint>
     <joint name="${prefix}wrist_3_joint" type="revolute">
@@ -310,5 +310,5 @@
          <safety_controller soft_lower_limit="${wrist_3_lower_limit + safety_pos_margin}" soft_upper_limit="${wrist_3_upper_limit - safety_pos_margin}" k_position="${safety_k_position}" k_velocity="0.0"/>
       </xacro:if>
-      <dynamics damping="0" friction="0"/>
+      <dynamics damping="5" friction="5"/>
     </joint>
     <!-- ROS-Industrial 'base' frame - base_link to UR 'Base' Coordinates transform -->

Commit message: added initial_positions yaml file to serve as an example

File: ur_description/urdf/ur.urdf.xacro (robot description, xacro)
@@ -18,4 +18,7 @@
    <xacro:arg name="use_fake_hardware" default="false" />
    <xacro:arg name="fake_sensor_commands" default="false" />
+   <!-- initial position -->
+   <xacro:arg name="initial_positions_file" default="$(find ur_description)/config/initial_positions.yaml"/>
+   <xacro:property name="initial_positions_file" default="$(arg initial_positions_file)"/>
    <!-- arm -->
    <xacro:ur_robot
@@ -30,4 +33,5 @@
      safety_k_position="$(arg safety_k_position)"
      use_fake_hardware="$(arg use_fake_hardware)"
-     fake_sensor_commands="$(arg fake_sensor_commands)" />
+     fake_sensor_commands="$(arg fake_sensor_commands)"
+     initial_positions="${load_yaml(initial_positions_file)}" />
 </robot>

Commit message: Add ft_sensor frame.

File: ur_description/urdf/ur.urdf.xacro (robot description, xacro)
@@ -25,7 +25,10 @@
    <!-- convert to property to use substitution in function -->
    <xacro:property name="initial_positions_file" default="$(arg initial_positions_file)"/>
+   <!-- create link fixed to the "world" -->
+   <link name="world" />
    <!-- arm -->
    <xacro:ur_robot
      prefix="$(arg prefix)"
+     parent="world"
      joint_limits_parameters_file="$(arg joint_limit_params)"
      kinematics_parameters_file="$(arg kinematics_params)"
@@ -40,4 +43,6 @@
      headless_mode="$(arg headless_mode)"
      initial_positions="${load_yaml(initial_positions_file)}"
-     ignition="$(arg ignition)" />
+     ignition="$(arg ignition)" >
+    <origin xyz="0 0 0" rpy="0 0 0" />          <!-- position robot in the world -->
+   </xacro:ur_robot>
 </robot>

File: ur_description/urdf/ur_macro.xacro (robot description, xacro)
@@ -46,4 +46,6 @@
   <xacro:macro name="ur_robot" params="
     prefix
+    parent
+    *origin
     joint_limits_parameters_file
     kinematics_parameters_file
@@ -209,4 +211,10 @@
       </xacro:cylinder_inertial>
     </link>
+    <!-- base_joint fixes base_link to the environment -->
+    <joint name="${prefix}base_joint" type="fixed">
+      <xacro:insert_block name="origin" />
+      <parent link="${parent}" />
+      <child link="${prefix}base_link" />
+    </joint>
     <!-- joints - main serial chain -->
     <joint name="${prefix}base_link-base_link_inertia" type="fixed">
@@ -291,4 +299,10 @@
       </xacro:if>
       <dynamics damping="5" friction="5"/>
+    </joint>
+    <link name="${prefix}ft_frame"/>
+    <joint name="${prefix}wrist_3_link-ft_frame" type="fixed">
+      <parent link="${prefix}wrist_3_link"/>
+      <child link="${prefix}ft_frame"/>
+      <origin xyz="0 0 0" rpy="${pi} 0 0"/>
     </joint>
     <!-- ROS-Industrial 'base' frame - base_link to UR 'Base' Coordinates transform -->
@@ -314,21 +328,15 @@
     <link name="${prefix}tool0"/>
     <joint name="${prefix}flange-tool0" type="fixed">
+      <parent link="${prefix}flange"/>
+      <child link="${prefix}tool0"/>
       <!-- default toolframe - X+ left, Y+ up, Z+ front -->
       <origin xyz="0 0 0" rpy="${pi/2.0} 0 ${pi/2.0}"/>
-      <parent link="${prefix}flange"/>
-      <child link="${prefix}tool0"/>
-    </joint>
-    <!-- Create a world link, and a fixed joint between world and base_link -->
-    <link name="world" />
-    <joint name="${prefix}world_joint"  type="fixed">
-      <origin xyz="0 0 0" rpy="0 0 0" />
-      <parent link="world"/>
-      <child link="${prefix}base_link"/>
     </joint>
     <!-- Ignition Gazebo -->
+    <!-- TODO(destogl): propagate `prefix` here down in the document, otherwise no multi-robot simulation is possible. -->
     <xacro:if value="${ignition}">
       <!-- Include Ignition Gazebo Plugins -->
       <xacro:include filename="ur_ignition_plugins.xacro" />
     </xacro:if>
-  </xacro:macro>
+    </xacro:macro>
 </robot>

Commit message: Organizational changes, docs and a little more tuning

File: ur_description/urdf/ur.urdf.xacro (robot description, xacro)
@@ -21,4 +21,6 @@
    <!-- initial position for fake hardware -->
    <xacro:arg name="initial_positions_file" default="$(find ur_description)/config/initial_positions.yaml"/>
+   <!-- Simulation parameter -->
+   <xacro:arg name="ignition" default="false" />
    <!-- convert to property to use substitution in function -->
    <xacro:property name="initial_positions_file" default="$(arg initial_positions_file)"/>
@@ -37,6 +39,5 @@
      fake_sensor_commands="$(arg fake_sensor_commands)"
      headless_mode="$(arg headless_mode)"
-     initial_positions="${load_yaml(initial_positions_file)}" />
-  <!-- Ignition -->
-  <xacro:include filename="ur_ignition_plugins.xacro" />
+     initial_positions="${load_yaml(initial_positions_file)}"
+     ignition="$(arg ignition)" />
 </robot>

File: ur_description/urdf/ur_ignition_plugins.xacro (robot description, xacro)
@@ -3,5 +3,5 @@
   <!-- Joint Controller Gains -->
   <xacro:property name="default_initial_position" value="0"/>
-  <xacro:property name="default_position_p_gain" value="3000"/>
+  <xacro:property name="default_position_p_gain" value="1500"/>
   <xacro:property name="default_position_d_gain" value="15"/>
   <xacro:property name="default_position_i_gain" value="1650"/>

File: ur_description/urdf/ur_macro.xacro (robot description, xacro)
@@ -57,4 +57,5 @@
     fake_sensor_commands:=false
     headless_mode:=false
+    ignition:=false
     initial_positions:=${dict(shoulder_pan_joint=0.0,shoulder_lift_joint=-1.57,elbow_joint=0.0,wrist_1_joint=-1.57,wrist_2_joint=0.0,wrist_3_joint=0.0)}">
     <!-- Load configuration data from the provided .yaml files -->
@@ -325,4 +326,8 @@
       <child link="${prefix}tool0"/>
     </joint>
+  <!-- Ignition Plugins -->
+  <xacro:if value="${ignition}">
+    <xacro:include filename="ur_ignition_plugins.xacro" />
+  </xacro:if>
   </xacro:macro>
 </robot>
