Commit message: replaced *origin with xyp rpy to set default values

File: ur_description/urdf/ur.urdf.xacro (robot description, xacro)
@@ -50,6 +50,7 @@
      initial_positions="${load_yaml(initial_positions_file)}"
      sim_gazebo="$(arg sim_gazebo)"
-     sim_ignition="$(arg sim_ignition)">
-     <origin xyz="$(arg xyz)" rpy="$(arg rpy)" />          <!-- position robot in the world; only used when joint_to_parent=true -->
+     sim_ignition="$(arg sim_ignition)"
+     xyz="$(arg xyz)" rpy="$(arg rpy)" > <!-- position robot in the world; only used when joint_to_parent=true -->
+     <!-- <origin xyz="$(arg xyz)" rpy="$(arg rpy)" />    -->
    </xacro:ur_robot>
     <xacro:if value="$(arg sim_gazebo)">

File: ur_description/urdf/ur_macro.xacro (robot description, xacro)
@@ -44,9 +44,12 @@
   <xacro:include filename="$(find ur_description)/urdf/inc/ur_transmissions.xacro" />
   <xacro:include filename="$(find ur_description)/urdf/inc/ur_common.xacro" />
+  <xacro:property name="default_xyz" default="0 0 0"/>
+  <xacro:property name="default_rpy" default="0 0 0"/>
   <xacro:macro name="ur_robot" params="
     prefix
-    parent
+    parent:=world
     joint_to_parent:=false
-    *origin
+    xyz:=${default_xyz}
+    rpy:=${default_rpy}
     joint_limits_parameters_file
     kinematics_parameters_file
@@ -238,5 +241,6 @@
     <xacro:if value="${joint_to_parent}">
       <joint name="${prefix}base_joint" type="fixed">
-        <xacro:insert_block name="origin" />
+        <!-- <xacro:insert_block name="origin" /> -->
+        <origin xyz="${xyz}" rpy="${rpy}" />
         <parent link="${parent}" />
         <child link="${prefix}base_link" />

Commit message: went back to old commit 2e5a31d(added get_mesh macro, updated gazebo simulation launch file, removed ur5 urdf files)

File: ur_description/urdf/ur.urdf.xacro (robot description, xacro)
@@ -18,9 +18,4 @@
    <xacro:arg name="sim_ignition" default="false" />
    <xacro:arg name="simulation_controllers" default="" />
-   <xacro:arg name="joint_to_parent" default="false" />
-   <xacro:arg name="create_link_world" default="false" />
-   <xacro:arg name="parent" default="world" />
-   <xacro:arg name="xyz" default="0 0 0" />
-   <xacro:arg name="rpy" default="0 0 0" />
    <!-- ros2_control related parameters -->
    <xacro:arg name="use_fake_hardware" default="false" />
@@ -29,13 +24,7 @@
    <xacro:arg name="initial_positions_file" default="$(find ur_description)/config/initial_positions.yaml"/>
    <xacro:property name="initial_positions_file" default="$(arg initial_positions_file)"/>
-   <xacro:if value="$(arg create_link_world)">
-     <!-- create link fixed to the "world" -->
-     <link name="world" />
-   </xacro:if>
    <!-- arm -->
    <xacro:ur_robot
      prefix="$(arg prefix)"
-     joint_to_parent="$(arg joint_to_parent)"
-     parent="$(arg parent)"
      joint_limits_parameters_file="$(arg joint_limit_params)"
      kinematics_parameters_file="$(arg kinematics_params)"
@@ -50,8 +39,5 @@
      initial_positions="${load_yaml(initial_positions_file)}"
      sim_gazebo="$(arg sim_gazebo)"
-     sim_ignition="$(arg sim_ignition)"
-     xyz="$(arg xyz)" rpy="$(arg rpy)" > <!-- position robot in the world; only used when joint_to_parent=true -->
-     <!-- <origin xyz="$(arg xyz)" rpy="$(arg rpy)" />    -->
-   </xacro:ur_robot>
+     sim_ignition="$(arg sim_ignition)"/>
     <xacro:if value="$(arg sim_gazebo)">
       <!-- Gazebo plugins -->

File: ur_description/urdf/ur_macro.xacro (robot description, xacro)
@@ -44,12 +44,6 @@
   <xacro:include filename="$(find ur_description)/urdf/inc/ur_transmissions.xacro" />
   <xacro:include filename="$(find ur_description)/urdf/inc/ur_common.xacro" />
-  <xacro:property name="default_xyz" default="0 0 0"/>
-  <xacro:property name="default_rpy" default="0 0 0"/>
   <xacro:macro name="ur_robot" params="
     prefix
-    parent:=world
-    joint_to_parent:=false
-    xyz:=${default_xyz}
-    rpy:=${default_rpy}
     joint_limits_parameters_file
     kinematics_parameters_file
@@ -238,13 +232,4 @@
       </xacro:cylinder_inertial>
     </link>
-    <!-- base_joint fixes base_link to the environment -->
-    <xacro:if value="${joint_to_parent}">
-      <joint name="${prefix}base_joint" type="fixed">
-        <!-- <xacro:insert_block name="origin" /> -->
-        <origin xyz="${xyz}" rpy="${rpy}" />
-        <parent link="${parent}" />
-        <child link="${prefix}base_link" />
-      </joint>
-    </xacro:if>
     <!-- joints - main serial chain -->
     <joint name="${prefix}base_link-base_link_inertia" type="fixed">
