Commit message: Some rewrapping and testing GPIO controller.

File: ur_description/urdf/ur.ros2_control.xacro (robot description, xacro)
@@ -1,5 +1,5 @@
 <?xml version="1.0"?>
 <robot xmlns:xacro="http://www.ros.org/wiki/xacro">
-  <xacro:macro name="ur5_system_position_only" params="name prefix
+  <xacro:macro name="ur_ros2_control" params="name prefix
     use_fake_hardware:=^|false fake_sensor_commands:=^|false
     script_filename output_recipe_filename
@@ -125,4 +125,102 @@
         <state_interface name="torque.z"/>
       </sensor>
+      <!-- NOTE The following are joints used only for testing with fake hardware and will chnage int the future -->
+      <joint name="speed_scaling">
+        <state_interface name="speed_scaling_factor"/>
+      </joint>
+      <joint name="gpio">
+        <command_interface name="standard_digital_output_cmd_0"/>
+        <command_interface name="standard_digital_output_cmd_1"/>
+        <command_interface name="standard_digital_output_cmd_2"/>
+        <command_interface name="standard_digital_output_cmd_3"/>
+        <command_interface name="standard_digital_output_cmd_4"/>
+        <command_interface name="standard_digital_output_cmd_5"/>
+        <command_interface name="standard_digital_output_cmd_6"/>
+        <command_interface name="standard_digital_output_cmd_7"/>
+        <command_interface name="standard_digital_output_cmd_8"/>
+        <command_interface name="standard_digital_output_cmd_9"/>
+        <command_interface name="standard_digital_output_cmd_10"/>
+        <command_interface name="standard_digital_output_cmd_11"/>
+        <command_interface name="standard_digital_output_cmd_12"/>
+        <command_interface name="standard_digital_output_cmd_13"/>
+        <command_interface name="standard_digital_output_cmd_14"/>
+        <command_interface name="standard_digital_output_cmd_15"/>
+        <command_interface name="standard_digital_output_cmd_16"/>
+        <command_interface name="standard_digital_output_cmd_17"/>
+        <command_interface name="standard_analog_output_cmd_0"/>
+        <command_interface name="standard_analog_output_cmd_1"/>
+        <command_interface name="io_async_success"/>
+        <command_interface name="speed_scaling_factor_cmd"/>
+        <command_interface name="scaling_async_success"/>
+        <state_interface name="digital_output_0"/>
+        <state_interface name="digital_output_1"/>
+        <state_interface name="digital_output_2"/>
+        <state_interface name="digital_output_3"/>
+        <state_interface name="digital_output_4"/>
+        <state_interface name="digital_output_5"/>
+        <state_interface name="digital_output_6"/>
+        <state_interface name="digital_output_7"/>
+        <state_interface name="digital_output_8"/>
+        <state_interface name="digital_output_9"/>
+        <state_interface name="digital_output_10"/>
+        <state_interface name="digital_output_11"/>
+        <state_interface name="digital_output_12"/>
+        <state_interface name="digital_output_13"/>
+        <state_interface name="digital_output_14"/>
+        <state_interface name="digital_output_15"/>
+        <state_interface name="digital_output_16"/>
+        <state_interface name="digital_output_17"/>
+        <state_interface name="digital_input_0"/>
+        <state_interface name="digital_input_1"/>
+        <state_interface name="digital_input_2"/>
+        <state_interface name="digital_input_3"/>
+        <state_interface name="digital_input_4"/>
+        <state_interface name="digital_input_5"/>
+        <state_interface name="digital_input_6"/>
+        <state_interface name="digital_input_7"/>
+        <state_interface name="digital_input_8"/>
+        <state_interface name="digital_input_9"/>
+        <state_interface name="digital_input_10"/>
+        <state_interface name="digital_input_11"/>
+        <state_interface name="digital_input_12"/>
+        <state_interface name="digital_input_13"/>
+        <state_interface name="digital_input_14"/>
+        <state_interface name="digital_input_15"/>
+        <state_interface name="digital_input_16"/>
+        <state_interface name="digital_input_17"/>
+        <state_interface name="standard_analog_output_0"/>
+        <state_interface name="standard_analog_output_1"/>
+        <state_interface name="standard_analog_input_0"/>
+        <state_interface name="standard_analog_input_1"/>
+        <state_interface name="analog_io_type_0"/>
+        <state_interface name="analog_io_type_1"/>
+        <state_interface name="analog_io_type_2"/>
+        <state_interface name="analog_io_type_3"/>
+        <state_interface name="tool_mode"/>
+        <state_interface name="tool_output_voltage"/>
+        <state_interface name="tool_output_current"/>
+        <state_interface name="tool_temperature"/>
+        <state_interface name="tool_analog_input_0"/>
+        <state_interface name="tool_analog_input_1"/>
+        <state_interface name="tool_analog_input_type_0"/>
+        <state_interface name="tool_analog_input_type_1"/>
+        <state_interface name="robot_mode"/>
+        <state_interface name="robot_status_bit_0"/>
+        <state_interface name="robot_status_bit_1"/>
+        <state_interface name="robot_status_bit_2"/>
+        <state_interface name="robot_status_bit_3"/>
+        <state_interface name="safety_mode"/>
+        <state_interface name="safety_status_bit_0"/>
+        <state_interface name="safety_status_bit_1"/>
+        <state_interface name="safety_status_bit_2"/>
+        <state_interface name="safety_status_bit_3"/>
+        <state_interface name="safety_status_bit_4"/>
+        <state_interface name="safety_status_bit_5"/>
+        <state_interface name="safety_status_bit_6"/>
+        <state_interface name="safety_status_bit_7"/>
+        <state_interface name="safety_status_bit_8"/>
+        <state_interface name="safety_status_bit_9"/>
+        <state_interface name="safety_status_bit_10"/>
+      </joint>
     </ros2_control>
   </xacro:macro>

Commit message: Added MoveIt configs and example launch file

File: ur_description/urdf/ur.ros2_control.xacro (robot description, xacro)
@@ -63,5 +63,5 @@
         <state_interface name="velocity"/>
         <state_interface name="effort"/>
-        <param name="initial_position">-1.57</param>  <!-- initial position for the FakeSystem -->
+        <param name="initial_position">0.0</param>  <!-- initial position for the FakeSystem -->
       </joint>
       <joint name="${prefix}elbow_joint">

File: ur_moveit_config/srdf/ur_macro.srdf.xacro (robot description, xacro)
@@ -14,11 +14,8 @@
       <chain base_link="${prefix}base_link" tip_link="${prefix}tool0" />
     </group>
-    <group name="${prefix}endeffector">
-      <link name="${prefix}tool0" />
-    </group>
     <!--GROUP STATES - Purpose - Define a named state for a particular group, in terms of joint values. This is useful to define states like 'folded arms'-->
     <group_state name="${prefix}home" group="${prefix}${name}_manipulator">
       <joint name="${prefix}elbow_joint" value="0" />
-      <joint name="${prefix}shoulder_lift_joint" value="0" />
+      <joint name="${prefix}shoulder_lift_joint" value="-1.5707" />
       <joint name="${prefix}shoulder_pan_joint" value="0" />
       <joint name="${prefix}wrist_1_joint" value="0" />
@@ -43,7 +40,6 @@
     </group_state>
     <!--END EFFECTOR - Purpose - Represent information about an end effector.-->
-    <end_effector name="${prefix}moveit_ee" parent_link="${prefix}tool0" group="${prefix}endeffector" />
     <!--VIRTUAL JOINT - Purpose - this element defines a virtual joint between a robot link and an external frame of reference (considered fixed with respect to the robot)-->
-    <virtual_joint name="${prefix}fixed_base" type="fixed" parent_frame="world" child_link="${prefix}base_link" />
+    <virtual_joint name="${prefix}fixed_base" type="floating" parent_frame="world" child_link="${prefix}base_link" />
     <!--DISABLE COLLISIONS - By default it is assumed that any link of the robot could potentially come into collision with any other link in the robot. This tag disables collision checking between a specified pair of links. -->
     <disable_collisions link1="${prefix}base_link" link2="${prefix}base_link_inertia" reason="Adjacent" />

Commit message: Add launch files and chnages for Gazebo simulation.

File: ur_description/urdf/ur.ros2_control.xacro (robot description, xacro)
@@ -3,4 +3,6 @@
   <xacro:macro name="ur_ros2_control" params="name prefix
     use_fake_hardware:=false fake_sensor_commands:=false
+    gazebo_sim:=false
+    gazebo_controllers:=MISSING_CONTROLLERS_YAML
     headless_mode:=false
     initial_positions:=${dict(shoulder_pan_joint=0.0,shoulder_lift_joint=-1.57,elbow_joint=0.0,wrist_1_joint=-1.57,wrist_2_joint=0.0,wrist_3_joint=0.0)}
@@ -8,4 +10,5 @@
     input_recipe_filename tf_prefix
     hash_kinematics robot_ip">
+  <xacro:unless value="${gazebo_sim}">
     <ros2_control name="${name}" type="system">
       <hardware>
@@ -239,4 +242,64 @@
       </joint>
     </ros2_control>
+  </xacro:unless>
+  <xacro:if value="${gazebo_sim}">
+    <!-- Gazebo plugins -->
+    <gazebo reference="world">
+    </gazebo>
+    <gazebo>
+      <plugin filename="libgazebo_ros2_control.so" name="gazebo_ros2_control">
+        <parameters>${gazebo_controllers}</parameters>
+      </plugin>
+    </gazebo>
+    <!-- TODO: Implement initial positions support in Gazebo - check ros-controls/gazebo_ros2_control#100 -->
+    <!-- ros2_control definition -->
+    <ros2_control name="${name}" type="system">
+      <hardware>
+        <plugin>gazebo_ros2_control/GazeboSystem</plugin>
+      </hardware>
+      <joint name="${prefix}shoulder_pan_joint">
+        <command_interface name="position"/>
+        <state_interface name="position"/>
+        <state_interface name="velocity"/>
+        <state_interface name="effort"/>
+        <param name="initial_position">${initial_positions['shoulder_pan_joint']}</param>  <!-- initial position for Gazebo -->
+      </joint>
+      <joint name="${prefix}shoulder_lift_joint">
+        <command_interface name="position"/>
+        <state_interface name="position"/>
+        <state_interface name="velocity"/>
+        <state_interface name="effort"/>
+        <param name="initial_position">${initial_positions['shoulder_lift_joint']}</param>  <!-- initial position for Gazebo -->
+      </joint>
+      <joint name="${prefix}elbow_joint">
+        <command_interface name="position"/>
+        <state_interface name="position"/>
+        <state_interface name="velocity"/>
+        <state_interface name="effort"/>
+        <param name="initial_position">${initial_positions['elbow_joint']}</param>  <!-- initial position for Gazebo -->
+      </joint>
+      <joint name="${prefix}wrist_1_joint">
+        <command_interface name="position"/>
+        <state_interface name="position"/>
+        <state_interface name="velocity"/>
+        <state_interface name="effort"/>
+        <param name="initial_position">${initial_positions['wrist_1_joint']}</param>  <!-- initial position for Gazebo -->
+      </joint>
+      <joint name="${prefix}wrist_2_joint">
+        <command_interface name="position"/>
+        <state_interface name="position"/>
+        <state_interface name="velocity"/>
+        <state_interface name="effort"/>
+        <param name="initial_position">${initial_positions['wrist_2_joint']}</param>  <!-- initial position for Gazebo -->
+      </joint>
+      <joint name="${prefix}wrist_3_joint">
+        <command_interface name="position"/>
+        <state_interface name="position"/>
+        <state_interface name="velocity"/>
+        <state_interface name="effort"/>
+        <param name="initial_position">${initial_positions['wrist_3_joint']}</param>  <!-- initial position for Gazebo -->
+      </joint>
+    </ros2_control>
+  </xacro:if>
   </xacro:macro>
 </robot>

File: ur_description/urdf/ur.urdf.xacro (robot description, xacro)
@@ -18,4 +18,6 @@
    <xacro:arg name="use_fake_hardware" default="false" />
    <xacro:arg name="fake_sensor_commands" default="false" />
+   <xacro:arg name="gazebo_sim" default="false" />
+   <xacro:arg name="gazebo_controllers" default="$(find ur_bringup)/config/ur_controllers.yaml" />
    <xacro:arg name="headless_mode" default="false" />
    <!-- initial position for fake hardware -->
@@ -29,4 +31,5 @@
    <!-- arm -->
    <xacro:ur_robot
+     name="$(arg name)"
      prefix="$(arg prefix)"
      parent="world"
@@ -41,4 +44,6 @@
      use_fake_hardware="$(arg use_fake_hardware)"
      fake_sensor_commands="$(arg fake_sensor_commands)"
+     gazebo_sim="$(arg gazebo_sim)"
+     gazebo_controllers="$(arg gazebo_controllers)"
      headless_mode="$(arg headless_mode)"
      initial_positions="${load_yaml(initial_positions_file)}"

File: ur_description/urdf/ur_macro.xacro (robot description, xacro)
@@ -45,4 +45,5 @@
   <xacro:include filename="$(find ur_description)/urdf/inc/ur_common.xacro" />
   <xacro:macro name="ur_robot" params="
+    name
     prefix
     parent
@@ -58,7 +59,9 @@
     use_fake_hardware:=false
     fake_sensor_commands:=false
+    gazebo_sim:=false
+    gazebo_controllers:=MISSING_CONTROLLERS_YAML
     headless_mode:=false
-    ignition:=false
-    initial_positions:=${dict(shoulder_pan_joint=0.0,shoulder_lift_joint=-1.57,elbow_joint=0.0,wrist_1_joint=-1.57,wrist_2_joint=0.0,wrist_3_joint=0.0)}">
+    initial_positions:=${dict(shoulder_pan_joint=0.0,shoulder_lift_joint=-1.57,elbow_joint=0.0,wrist_1_joint=-1.57,wrist_2_joint=0.0,wrist_3_joint=0.0)}
+    ignition:=false">
     <!-- Load configuration data from the provided .yaml files -->
     <xacro:read_model_data
@@ -76,9 +79,11 @@
     <!-- ros2 control instance -->
     <xacro:ur_ros2_control
-      name="URPositionHardwareInterface" prefix="${prefix}"
+      name="${name}" prefix="${prefix}"
       use_fake_hardware="$(arg use_fake_hardware)"
+      fake_sensor_commands="$(arg fake_sensor_commands)"
+      gazebo_sim="$(arg gazebo_sim)"
+      gazebo_controllers="$(arg gazebo_controllers)"
+      headless_mode="$(arg headless_mode)"
       initial_positions="${initial_positions}"
-      fake_sensor_commands="$(arg fake_sensor_commands)"
-      headless_mode="$(arg headless_mode)"
       script_filename="$(arg script_filename)"
       output_recipe_filename="$(arg output_recipe_filename)"
@@ -96,5 +101,5 @@
         <origin xyz="0 0 0" rpy="0 0 ${pi}"/>
         <geometry>
-          <mesh filename="${base_visual_mesh}"/>
+          <mesh filename="file://$(find ur_description)/meshes/${base_visual_mesh}"/>
         </geometry>
       </visual>
@@ -102,5 +107,5 @@
         <origin xyz="0 0 0" rpy="0 0 ${pi}"/>
         <geometry>
-          <mesh filename="${base_collision_mesh}"/>
+          <mesh filename="file://$(find ur_description)/meshes/${base_collision_mesh}"/>
         </geometry>
       </collision>
@@ -113,5 +118,5 @@
         <origin xyz="0 0 0" rpy="0 0 ${pi}"/>
         <geometry>
-          <mesh filename="${shoulder_visual_mesh}"/>
+          <mesh filename="file://$(find ur_description)/meshes/${shoulder_visual_mesh}"/>
         </geometry>
       </visual>
@@ -119,5 +124,5 @@
         <origin xyz="0 0 0" rpy="0 0 ${pi}"/>
         <geometry>
-          <mesh filename="${shoulder_collision_mesh}"/>
+          <mesh filename="file://$(find ur_description)/meshes/${shoulder_collision_mesh}"/>
         </geometry>
       </collision>
@@ -130,5 +135,5 @@
         <origin xyz="0 0 ${shoulder_offset}" rpy="${pi/2} 0 ${-pi/2}"/>
         <geometry>
-          <mesh filename="${upper_arm_visual_mesh}"/>
+          <mesh filename="file://$(find ur_description)/meshes/${upper_arm_visual_mesh}"/>
         </geometry>
       </visual>
@@ -136,5 +141,5 @@
         <origin xyz="0 0 ${shoulder_offset}" rpy="${pi/2} 0 ${-pi/2}"/>
         <geometry>
-          <mesh filename="${upper_arm_collision_mesh}"/>
+          <mesh filename="file://$(find ur_description)/meshes/${upper_arm_collision_mesh}"/>
         </geometry>
       </collision>
@@ -147,5 +152,5 @@
         <origin xyz="0 0 ${elbow_offset}" rpy="${pi/2} 0 ${-pi/2}"/>
         <geometry>
-          <mesh filename="${forearm_visual_mesh}"/>
+          <mesh filename="file://$(find ur_description)/meshes/${forearm_visual_mesh}"/>
         </geometry>
       </visual>
@@ -153,5 +158,5 @@
         <origin xyz="0 0 ${elbow_offset}" rpy="${pi/2} 0 ${-pi/2}"/>
         <geometry>
-          <mesh filename="${forearm_collision_mesh}"/>
+          <mesh filename="file://$(find ur_description)/meshes/${forearm_collision_mesh}"/>
         </geometry>
       </collision>
@@ -164,5 +169,5 @@
         <origin xyz="0 0 ${wrist_1_visual_offset}" rpy="${pi/2} 0 0"/>
         <geometry>
-          <mesh filename="${wrist_1_visual_mesh}"/>
+          <mesh filename="file://$(find ur_description)/meshes/${wrist_1_visual_mesh}"/>
         </geometry>
       </visual>
@@ -170,5 +175,5 @@
         <origin xyz="0 0 ${wrist_1_visual_offset}" rpy="${pi/2} 0 0"/>
         <geometry>
-          <mesh filename="${wrist_1_collision_mesh}"/>
+          <mesh filename="file://$(find ur_description)/meshes/${wrist_1_collision_mesh}"/>
         </geometry>
       </collision>
@@ -181,5 +186,5 @@
         <origin xyz="0 0 ${wrist_2_visual_offset}" rpy="0 0 0"/>
         <geometry>
-          <mesh filename="${wrist_2_visual_mesh}"/>
+          <mesh filename="file://$(find ur_description)/meshes/${wrist_2_visual_mesh}"/>
         </geometry>
       </visual>
@@ -187,5 +192,5 @@
         <origin xyz="0 0 ${wrist_2_visual_offset}" rpy="0 0 0"/>
         <geometry>
-          <mesh filename="${wrist_2_collision_mesh}"/>
+          <mesh filename="file://$(find ur_description)/meshes/${wrist_2_collision_mesh}"/>
         </geometry>
       </collision>
@@ -198,5 +203,5 @@
         <origin xyz="0 0 ${wrist_3_visual_offset}" rpy="${pi/2} 0 0"/>
         <geometry>
-          <mesh filename="${wrist_3_visual_mesh}"/>
+          <mesh filename="file://$(find ur_description)/meshes/${wrist_3_visual_mesh}"/>
         </geometry>
       </visual>
@@ -204,5 +209,5 @@
         <origin xyz="0 0 ${wrist_3_visual_offset}" rpy="${pi/2} 0 0"/>
         <geometry>
-          <mesh filename="${wrist_3_collision_mesh}"/>
+          <mesh filename="file://$(find ur_description)/meshes/${wrist_3_collision_mesh}"/>
         </geometry>
       </collision>
