Commit message: Optimize simulation files and add ignition to them too.

File: ur_description/urdf/ur.ros2_control.xacro (robot description, xacro)
@@ -4,5 +4,5 @@
     use_fake_hardware:=false fake_sensor_commands:=false
     gazebo_sim:=false
-    gazebo_controllers:=MISSING_CONTROLLERS_YAML
+    ignition_sim:=false
     headless_mode:=false
     initial_positions:=${dict(shoulder_pan_joint=0.0,shoulder_lift_joint=-1.57,elbow_joint=0.0,wrist_1_joint=-1.57,wrist_2_joint=0.0,wrist_3_joint=0.0)}
@@ -10,7 +10,12 @@
     input_recipe_filename tf_prefix
     hash_kinematics robot_ip">
-  <xacro:unless value="${gazebo_sim}">
     <ros2_control name="${name}" type="system">
       <hardware>
+        <xacro:if value="${gazebo_sim}">
+          <plugin>gazebo_ros2_control/GazeboSystem</plugin>
+        </xacro:if>
+        <xacro:if value="${ignition_sim}">
+          <plugin>ignition_ros2_control/IgnitionSystem</plugin>
+        </xacro:if>
         <xacro:if value="${use_fake_hardware}">
           <plugin>fake_components/GenericSystem</plugin>
@@ -18,5 +23,5 @@
           <param name="state_following_offset">0.0</param>
         </xacro:if>
-        <xacro:unless value="${use_fake_hardware}">
+        <xacro:unless value="${use_fake_hardware or gazebo_sim or ignition_sim}">
           <plugin>ur_robot_driver/URPositionHardwareInterface</plugin>
           <param name="robot_ip">${robot_ip}</param>
@@ -127,4 +132,5 @@
         <param name="initial_position">${initial_positions['wrist_3_joint']}</param>  <!-- initial position for the FakeSystem -->
       </joint>
+    <xacro:unless value="${gazebo_sim or ignition_sim}">
       <sensor name="tcp_fts_sensor">
         <state_interface name="force.x"/>
@@ -243,63 +249,4 @@
     </ros2_control>
   </xacro:unless>
-  <xacro:if value="${gazebo_sim}">
-    <!-- Gazebo plugins -->
-    <gazebo reference="world">
-    </gazebo>
-    <gazebo>
-      <plugin filename="libgazebo_ros2_control.so" name="gazebo_ros2_control">
-        <parameters>${gazebo_controllers}</parameters>
-      </plugin>
-    </gazebo>
-    <!-- TODO: Implement initial positions support in Gazebo - check ros-controls/gazebo_ros2_control#100 -->
-    <!-- ros2_control definition -->
-    <ros2_control name="${name}" type="system">
-      <hardware>
-        <plugin>gazebo_ros2_control/GazeboSystem</plugin>
-      </hardware>
-      <joint name="${prefix}shoulder_pan_joint">
-        <command_interface name="position"/>
-        <state_interface name="position"/>
-        <state_interface name="velocity"/>
-        <state_interface name="effort"/>
-        <param name="initial_position">${initial_positions['shoulder_pan_joint']}</param>  <!-- initial position for Gazebo -->
-      </joint>
-      <joint name="${prefix}shoulder_lift_joint">
-        <command_interface name="position"/>
-        <state_interface name="position"/>
-        <state_interface name="velocity"/>
-        <state_interface name="effort"/>
-        <param name="initial_position">${initial_positions['shoulder_lift_joint']}</param>  <!-- initial position for Gazebo -->
-      </joint>
-      <joint name="${prefix}elbow_joint">
-        <command_interface name="position"/>
-        <state_interface name="position"/>
-        <state_interface name="velocity"/>
-        <state_interface name="effort"/>
-        <param name="initial_position">${initial_positions['elbow_joint']}</param>  <!-- initial position for Gazebo -->
-      </joint>
-      <joint name="${prefix}wrist_1_joint">
-        <command_interface name="position"/>
-        <state_interface name="position"/>
-        <state_interface name="velocity"/>
-        <state_interface name="effort"/>
-        <param name="initial_position">${initial_positions['wrist_1_joint']}</param>  <!-- initial position for Gazebo -->
-      </joint>
-      <joint name="${prefix}wrist_2_joint">
-        <command_interface name="position"/>
-        <state_interface name="position"/>
-        <state_interface name="velocity"/>
-        <state_interface name="effort"/>
-        <param name="initial_position">${initial_positions['wrist_2_joint']}</param>  <!-- initial position for Gazebo -->
-      </joint>
-      <joint name="${prefix}wrist_3_joint">
-        <command_interface name="position"/>
-        <state_interface name="position"/>
-        <state_interface name="velocity"/>
-        <state_interface name="effort"/>
-        <param name="initial_position">${initial_positions['wrist_3_joint']}</param>  <!-- initial position for Gazebo -->
-      </joint>
-    </ros2_control>
-  </xacro:if>
   </xacro:macro>
 </robot>

File: ur_description/urdf/ur.urdf.xacro (robot description, xacro)
@@ -18,11 +18,11 @@
    <xacro:arg name="use_fake_hardware" default="false" />
    <xacro:arg name="fake_sensor_commands" default="false" />
-   <xacro:arg name="gazebo_sim" default="false" />
-   <xacro:arg name="gazebo_controllers" default="$(find ur_bringup)/config/ur_controllers.yaml" />
    <xacro:arg name="headless_mode" default="false" />
    <!-- initial position for fake hardware -->
    <xacro:arg name="initial_positions_file" default="$(find ur_description)/config/initial_positions.yaml"/>
    <!-- Simulation parameter -->
-   <xacro:arg name="ignition" default="false" />
+   <xacro:arg name="gazebo_sim" default="false" />
+   <xacro:arg name="ignition_sim" default="false" />
+   <xacro:arg name="simulation_controllers" default="$(find ur_bringup)/config/ur_controllers.yaml" />
    <!-- convert to property to use substitution in function -->
    <xacro:property name="initial_positions_file" default="$(arg initial_positions_file)"/>
@@ -44,10 +44,30 @@
      use_fake_hardware="$(arg use_fake_hardware)"
      fake_sensor_commands="$(arg fake_sensor_commands)"
-     gazebo_sim="$(arg gazebo_sim)"
-     gazebo_controllers="$(arg gazebo_controllers)"
      headless_mode="$(arg headless_mode)"
      initial_positions="${load_yaml(initial_positions_file)}"
-     ignition="$(arg ignition)" >
+     gazebo_sim="$(arg gazebo_sim)"
+     ignition_sim="$(arg ignition_sim)" >
     <origin xyz="0 0 0" rpy="0 0 0" />          <!-- position robot in the world -->
    </xacro:ur_robot>
+   <xacro:if value="$(arg gazebo_sim)">
+     <!-- Gazebo plugins -->
+     <gazebo reference="world">
+     </gazebo>
+     <gazebo>
+       <plugin filename="libgazebo_ros2_control.so" name="gazebo_ros2_control">
+         <parameters>$(arg simulation_controllers)</parameters>
+       </plugin>
+     </gazebo>
+   </xacro:if>
+   <xacro:if value="$(arg ignition_sim)">
+     <!-- Gazebo plugins -->
+     <gazebo reference="world">
+     </gazebo>
+     <gazebo>
+       <plugin filename="libignition_ros2_control-system.so" name="ignition_ros2_control::IgnitionROS2ControlPlugin">
+         <parameters>$(arg simulation_controllers)</parameters>
+         <controller_manager_node_name>$(arg prefix)controller_manager</controller_manager_node_name>
+       </plugin>
+     </gazebo>
+   </xacro:if>
 </robot>

File: ur_description/urdf/ur_macro.xacro (robot description, xacro)
@@ -60,8 +60,7 @@
     fake_sensor_commands:=false
     gazebo_sim:=false
-    gazebo_controllers:=MISSING_CONTROLLERS_YAML
+    ignition_sim:=false
     headless_mode:=false
-    initial_positions:=${dict(shoulder_pan_joint=0.0,shoulder_lift_joint=-1.57,elbow_joint=0.0,wrist_1_joint=-1.57,wrist_2_joint=0.0,wrist_3_joint=0.0)}
-    ignition:=false">
+    initial_positions:=${dict(shoulder_pan_joint=0.0,shoulder_lift_joint=-1.57,elbow_joint=0.0,wrist_1_joint=-1.57,wrist_2_joint=0.0,wrist_3_joint=0.0)}">
     <!-- Load configuration data from the provided .yaml files -->
     <xacro:read_model_data
@@ -83,5 +82,5 @@
       fake_sensor_commands="$(arg fake_sensor_commands)"
       gazebo_sim="$(arg gazebo_sim)"
-      gazebo_controllers="$(arg gazebo_controllers)"
+      ignition_sim="$(arg ignition_sim)"
       headless_mode="$(arg headless_mode)"
       initial_positions="${initial_positions}"

Commit message: Foxy controller stopper (#324)
* Added controller stopper node (Backport #309)
* Add state interface to ur_description
* Async tasks to seperate thread and initialized state interface (Backport parts of #206) (#372)
* Add system_interface initialized

Co-authored-by: Mads Holm Peters <79145214+urmahp@users.noreply.github.com>

File: ur_description/urdf/ur.ros2_control.xacro (robot description, xacro)
@@ -229,5 +229,9 @@
         <state_interface name="safety_status_bit_9"/>
         <state_interface name="safety_status_bit_10"/>
-      </joint>
+        <state_interface name="program_running"/>
+      </joint>
+      <gpio name="system_interface">
+        <state_interface name="initialized"/>
+      </gpio>
     </ros2_control>
   </xacro:macro>

Commit message: changed description for gazebo simulation

File: ur_description/urdf/ur.ros2_control.xacro (robot description, xacro)
@@ -9,4 +9,7 @@
     <ros2_control name="${name}" type="system">
       <hardware>
+        <xacro:if value="$(arg is_sim)">
+          <plugin>gazebo_ros2_control/GazeboSystem</plugin>
+        </xacro:if>
         <xacro:if value="${use_fake_hardware}">
           <plugin>fake_components/GenericSystem</plugin>

File: ur_description/urdf/ur_macro.xacro (robot description, xacro)
@@ -73,7 +73,7 @@
     <xacro:ur_ros2_control
       name="URPositionHardwareInterface" prefix="${prefix}"
-      use_fake_hardware="$(arg use_fake_hardware)"
+      use_fake_hardware="${use_fake_hardware}"
       initial_positions="${initial_positions}"
-      fake_sensor_commands="$(arg fake_sensor_commands)"
+      fake_sensor_commands="${fake_sensor_commands}"
       script_filename="$(arg script_filename)"
       output_recipe_filename="$(arg output_recipe_filename)"
@@ -91,5 +91,5 @@
         <origin xyz="0 0 0" rpy="0 0 ${pi}"/>
         <geometry>
-          <mesh filename="${base_visual_mesh}"/>
+          <mesh filename="file://$(find ${base_visual_mesh['package']})/${base_visual_mesh['path']}"/>
         </geometry>
         <material name="${base_visual_material_name}">
@@ -100,5 +100,5 @@
         <origin xyz="0 0 0" rpy="0 0 ${pi}"/>
         <geometry>
-          <mesh filename="${base_collision_mesh}"/>
+          <mesh filename="file://$(find ${base_collision_mesh['package']})/${base_collision_mesh['path']}"/>
         </geometry>
       </collision>
@@ -111,5 +111,5 @@
         <origin xyz="0 0 0" rpy="0 0 ${pi}"/>
         <geometry>
-          <mesh filename="${shoulder_visual_mesh}"/>
+          <mesh filename="file://$(find ${shoulder_visual_mesh['package']})/${shoulder_visual_mesh['path']}"/>
         </geometry>
         <material name="${shoulder_visual_material_name}">
@@ -120,5 +120,5 @@
         <origin xyz="0 0 0" rpy="0 0 ${pi}"/>
         <geometry>
-          <mesh filename="${shoulder_collision_mesh}"/>
+          <mesh filename="file://$(find ${shoulder_collision_mesh['package']})/${shoulder_collision_mesh['path']}"/>
         </geometry>
       </collision>
@@ -131,5 +131,5 @@
         <origin xyz="0 0 ${shoulder_offset}" rpy="${pi/2} 0 ${-pi/2}"/>
         <geometry>
-          <mesh filename="${upper_arm_visual_mesh}"/>
+          <mesh filename="file://$(find ${upper_arm_visual_mesh['package']})/${upper_arm_visual_mesh['path']}"/>
         </geometry>
         <material name="${upper_arm_visual_material_name}">
@@ -140,5 +140,5 @@
         <origin xyz="0 0 ${shoulder_offset}" rpy="${pi/2} 0 ${-pi/2}"/>
         <geometry>
-          <mesh filename="${upper_arm_collision_mesh}"/>
+          <mesh filename="file://$(find ${upper_arm_collision_mesh['package']})/${upper_arm_collision_mesh['path']}"/>
         </geometry>
       </collision>
@@ -151,5 +151,5 @@
         <origin xyz="0 0 ${elbow_offset}" rpy="${pi/2} 0 ${-pi/2}"/>
         <geometry>
-          <mesh filename="${forearm_visual_mesh}"/>
+          <mesh filename="file://$(find ${forearm_visual_mesh['package']})/${forearm_visual_mesh['path']}"/>
         </geometry>
         <material name="${forearm_visual_material_name}">
@@ -160,5 +160,5 @@
         <origin xyz="0 0 ${elbow_offset}" rpy="${pi/2} 0 ${-pi/2}"/>
         <geometry>
-          <mesh filename="${forearm_collision_mesh}"/>
+          <mesh filename="file://$(find ${forearm_collision_mesh['package']})/${forearm_collision_mesh['path']}"/>
         </geometry>
       </collision>
@@ -171,5 +171,5 @@
         <origin xyz="0 0 ${wrist_1_visual_offset}" rpy="${pi/2} 0 0"/>
         <geometry>
-          <mesh filename="${wrist_1_visual_mesh}"/>
+          <mesh filename="file://$(find ${wrist_1_visual_mesh['package']})/${wrist_1_visual_mesh['path']}"/>
         </geometry>
         <material name="${wrist_1_visual_material_name}">
@@ -180,5 +180,5 @@
         <origin xyz="0 0 ${wrist_1_visual_offset}" rpy="${pi/2} 0 0"/>
         <geometry>
-          <mesh filename="${wrist_1_collision_mesh}"/>
+          <mesh filename="file://$(find ${wrist_1_collision_mesh['package']})/${wrist_1_collision_mesh['path']}"/>
         </geometry>
       </collision>
@@ -191,5 +191,5 @@
         <origin xyz="0 0 ${wrist_2_visual_offset}" rpy="0 0 0"/>
         <geometry>
-          <mesh filename="${wrist_2_visual_mesh}"/>
+          <mesh filename="file://$(find ${wrist_2_visual_mesh['package']})/${wrist_2_visual_mesh['path']}"/>
         </geometry>
         <material name="${wrist_2_visual_material_name}">
@@ -200,5 +200,5 @@
         <origin xyz="0 0 ${wrist_2_visual_offset}" rpy="0 0 0"/>
         <geometry>
-          <mesh filename="${wrist_2_collision_mesh}"/>
+          <mesh filename="file://$(find ${wrist_2_collision_mesh['package']})/${wrist_2_collision_mesh['path']}"/>
         </geometry>
       </collision>
@@ -211,5 +211,5 @@
         <origin xyz="0 0 ${wrist_3_visual_offset}" rpy="${pi/2} 0 0"/>
         <geometry>
-          <mesh filename="${wrist_3_visual_mesh}"/>
+          <mesh filename="file://$(find ${wrist_3_visual_mesh['package']})/${wrist_3_visual_mesh['path']}"/>
         </geometry>
         <material name="${wrist_3_visual_material_name}">
@@ -220,5 +220,5 @@
         <origin xyz="0 0 ${wrist_3_visual_offset}" rpy="${pi/2} 0 0"/>
         <geometry>
-          <mesh filename="${wrist_3_collision_mesh}"/>
+          <mesh filename="file://$(find ${wrist_3_collision_mesh['package']})/${wrist_3_collision_mesh['path']}"/>
         </geometry>
       </collision>
