Commit message: added get_mesh macro and ignition simulation

File: ur_description/urdf/inc/ur_common.xacro (robot description, xacro)
@@ -20,5 +20,23 @@
     </inertial>
   </xacro:macro>
-  <xacro:macro name="read_model_data" params="joint_limits_parameters_file kinematics_parameters_file physical_parameters_file visual_parameters_file">
+  <xacro:macro name="get_visual_params" params="name:=^ type:=^" >
+    <xacro:property name="visual_params" value="${sec_mesh_files[name][type]}" scope="parent"/>
+  </xacro:macro>
+  <!-- Simplification of getting meshes. Available types can be seen in the visual_parameters.yaml (At the time of writing: visual, collision) -->
+  <xacro:macro name="get_mesh_path" params="name:=^ type:=^" >
+    <xacro:get_visual_params />
+    <xacro:if value="${force_abs_paths}">
+      <xacro:property name="mesh" value="file://$(find ${visual_params['mesh']['package']})/${visual_params['mesh']['path']}" scope="parent"/>
+    </xacro:if>
+    <xacro:unless value="${force_abs_paths}">
+      <xacro:property name="mesh" value="package://${visual_params['mesh']['package']}/${visual_params['mesh']['path']}" scope="parent"/>
+    </xacro:unless>
+  </xacro:macro>
+  <xacro:macro name="get_mesh" params="name type" >
+    <xacro:get_mesh_path/>
+    <mesh filename="${mesh}"/>
+  </xacro:macro>
+  <xacro:macro name="read_model_data" params="joint_limits_parameters_file kinematics_parameters_file physical_parameters_file visual_parameters_file force_abs_paths">
+    <xacro:property name="force_abs_paths" value="${force_abs_paths}" scope="parent"/>
     <!-- Read .yaml files from disk, load content into properties -->
     <xacro:property name="config_joint_limit_parameters" value="${load_yaml(joint_limits_parameters_file)}"/>
@@ -31,5 +49,5 @@
     <xacro:property name="sec_offsets" value="${config_physical_parameters['offsets']}"/>
     <xacro:property name="sec_inertia_parameters" value="${config_physical_parameters['inertia_parameters']}" />
-    <xacro:property name="sec_mesh_files" value="${config_visual_parameters['mesh_files']}" />
+    <xacro:property name="sec_mesh_files" value="${config_visual_parameters['mesh_files']}" scope="parent"/>
     <xacro:property name="sec_kinematics" value="${config_kinematics_parameters['kinematics']}" />
     <!-- JOINTS LIMIT PARAMETERS -->

File: ur_description/urdf/ur.ros2_control.xacro (robot description, xacro)
@@ -7,9 +7,13 @@
     input_recipe_filename tf_prefix
     hash_kinematics robot_ip
-    is_sim:=false">
+    sim_gazebo:=false
+    sim_ignition:=false">
     <ros2_control name="${name}" type="system">
       <hardware>
-        <xacro:if value="${is_sim}">
+        <xacro:if value="${sim_gazebo}">
           <plugin>gazebo_ros2_control/GazeboSystem</plugin>
+        </xacro:if>
+        <xacro:if value="${sim_ignition}">
+          <plugin>ign_ros2_control/IgnitionSystem</plugin>
         </xacro:if>
         <xacro:if value="${use_fake_hardware}">

File: ur_description/urdf/ur.urdf.xacro (robot description, xacro)
@@ -1,4 +1,5 @@
 <?xml version="1.0"?>
-<robot xmlns:xacro="http://wiki.ros.org/xacro" name="$(arg name)">
+<!-- <robot xmlns:xacro="http://wiki.ros.org/xacro" name="$(arg name)"> -->
+<robot xmlns:xacro="http://wiki.ros.org/xacro" name="">
    <!-- robot name parameter -->
    <xacro:arg name="name" default="ur"/>
@@ -15,5 +16,7 @@
    <xacro:arg name="safety_pos_margin" default="0.15"/>
    <xacro:arg name="safety_k_position" default="20"/>
-   <xacro:arg name="is_sim" default="false"/>
+   <xacro:arg name="sim_gazebo" default="false" />
+   <xacro:arg name="sim_ignition" default="false" />
+   <xacro:arg name="simulation_controllers" default="" />
    <!-- ros2_control related parameters -->
    <xacro:arg name="use_fake_hardware" default="false" />
@@ -36,11 +39,26 @@
      fake_sensor_commands="$(arg fake_sensor_commands)"
      initial_positions="${load_yaml(initial_positions_file)}"
-     is_sim="$(arg is_sim)"/>
-   <xacro:if value="$(arg is_sim)">
-     <gazebo>
-       <plugin name="$(arg prefix)gazebo_ros2_control" filename="libgazebo_ros2_control.so">
-         <parameters>$(arg gazebo_controllers)</parameters>
-       </plugin>
-     </gazebo>
-   </xacro:if>
+     sim_gazebo="$(arg sim_gazebo)"
+     sim_ignition="$(arg sim_ignition)"/>
+    <xacro:if value="$(arg sim_gazebo)">
+      <!-- Gazebo plugins -->
+      <gazebo reference="world">
+      </gazebo>
+      <gazebo>
+        <plugin filename="libgazebo_ros2_control.so" name="gazebo_ros2_control">
+          <parameters>$(arg simulation_controllers)</parameters>
+        </plugin>
+      </gazebo>
+    </xacro:if>
+    <xacro:if value="$(arg sim_ignition)">
+      <!-- Gazebo plugins -->
+      <gazebo reference="world">
+      </gazebo>
+      <gazebo>
+        <plugin filename="libign_ros2_control-system.so" name="ign_ros2_control::IgnitionROS2ControlPlugin">
+          <parameters>$(arg simulation_controllers)</parameters>
+          <controller_manager_node_name>$(arg prefix)controller_manager</controller_manager_node_name>
+        </plugin>
+      </gazebo>
+    </xacro:if>
 </robot>

File: ur_description/urdf/ur_macro.xacro (robot description, xacro)
@@ -56,5 +56,6 @@
     use_fake_hardware:=false
     fake_sensor_commands:=false
-    is_sim:=false
+    sim_gazebo:=false
+    sim_ignition:=false
     initial_positions:=${dict(shoulder_pan_joint=0.0,shoulder_lift_joint=-1.57,elbow_joint=0.0,wrist_1_joint=-1.57,wrist_2_joint=0.0,wrist_3_joint=0.0)}">
     <!-- Load configuration data from the provided .yaml files -->
@@ -63,5 +64,6 @@
       kinematics_parameters_file="${kinematics_parameters_file}"
       physical_parameters_file="${physical_parameters_file}"
-      visual_parameters_file="${visual_parameters_file}"/>
+      visual_parameters_file="${visual_parameters_file}"
+      force_abs_paths="${sim_gazebo or sim_ignition}"/>
     <!-- Data files required by the UR driver -->
     <xacro:arg name="script_filename" default="$(find ur_robot_driver)/resources/ros_control.urscript"/>
@@ -83,5 +85,6 @@
       hash_kinematics="${kinematics_hash}"
       robot_ip="$(arg robot_ip)"
-      is_sim="${is_sim}"/>
+      sim_gazebo="${sim_gazebo}"
+      sim_ignition="${sim_ignition}"/>
     <!-- Add URDF transmission elements (for ros_control) -->
     <!--<xacro:ur_arm_transmission prefix="${prefix}" hw_interface="${transmission_hw_interface}" />-->
