Commit message: Add tf_prefix support to MoveIt SRDF
The URDF supports a tf_prefix parameter to prefix all link and joint
names, but the MoveIt SRDF hardcoded the unprefixed names. As a result,
using a non-empty tf_prefix caused MoveIt to fail building the
ur_manipulator group because the referenced joints/links did not exist
in the URDF.

Thread a tf_prefix parameter (default empty, fully backward compatible)
through the SRDF macro, its wrapper, and the ur_moveit.launch.py launch
file so the SRDF link/joint references match the generated URDF.

Closes #1937

File: ur_moveit_config/srdf/ur.srdf.xacro (robot description, xacro)
@@ -3,5 +3,7 @@
   <!-- robot name parameter -->
   <xacro:arg name="name" default="ur"/>
+  <!-- parameters -->
+  <xacro:arg name="tf_prefix" default="" />
   <xacro:include filename="$(find ur_moveit_config)/srdf/ur_macro.srdf.xacro"/>
-  <xacro:ur_srdf/>
+  <xacro:ur_srdf tf_prefix="$(arg tf_prefix)"/>
 </robot>

File: ur_moveit_config/srdf/ur_macro.srdf.xacro (robot description, xacro)
@@ -5,5 +5,5 @@
     A URDF file must exist for this robot as well, where the joints and the links that are referenced are defined
 -->
-  <xacro:macro name="ur_srdf" params="">
+  <xacro:macro name="ur_srdf" params="tf_prefix=''">
     <!--GROUPS - Representation of a set of joints and links. This can be useful for specifying DOF to plan for, defining arms, end effectors, etc-->
     <!--LINKS - When a link is specified, the parent joint of that link (if it exists) is automatically included-->
@@ -12,45 +12,45 @@
     <!--SUBGROUPS - Groups can also be formed by referencing to already defined group names-->
     <group name="ur_manipulator">
-      <chain base_link="base_link" tip_link="tool0" />
+      <chain base_link="${tf_prefix}base_link" tip_link="${tf_prefix}tool0" />
     </group>
     <!--GROUP STATES - Purpose - Define a named state for a particular group, in terms of joint values. This is useful to define states like 'folded arms'-->
     <group_state name="home" group="ur_manipulator">
-      <joint name="elbow_joint" value="0" />
-      <joint name="shoulder_lift_joint" value="-1.5707" />
-      <joint name="shoulder_pan_joint" value="0" />
-      <joint name="wrist_1_joint" value="0" />
-      <joint name="wrist_2_joint" value="0" />
-      <joint name="wrist_3_joint" value="0" />
+      <joint name="${tf_prefix}elbow_joint" value="0" />
+      <joint name="${tf_prefix}shoulder_lift_joint" value="-1.5707" />
+      <joint name="${tf_prefix}shoulder_pan_joint" value="0" />
+      <joint name="${tf_prefix}wrist_1_joint" value="0" />
+      <joint name="${tf_prefix}wrist_2_joint" value="0" />
+      <joint name="${tf_prefix}wrist_3_joint" value="0" />
     </group_state>
     <group_state name="up" group="ur_manipulator">
-      <joint name="elbow_joint" value="0" />
-      <joint name="shoulder_lift_joint" value="-1.5707" />
-      <joint name="shoulder_pan_joint" value="0" />
-      <joint name="wrist_1_joint" value="-1.5707" />
-      <joint name="wrist_2_joint" value="0" />
-      <joint name="wrist_3_joint" value="0" />
+      <joint name="${tf_prefix}elbow_joint" value="0" />
+      <joint name="${tf_prefix}shoulder_lift_joint" value="-1.5707" />
+      <joint name="${tf_prefix}shoulder_pan_joint" value="0" />
+      <joint name="${tf_prefix}wrist_1_joint" value="-1.5707" />
+      <joint name="${tf_prefix}wrist_2_joint" value="0" />
+      <joint name="${tf_prefix}wrist_3_joint" value="0" />
     </group_state>
     <group_state name="test_configuration" group="ur_manipulator">
-      <joint name="elbow_joint" value="1.4" />
-      <joint name="shoulder_lift_joint" value="-1.62" />
-      <joint name="shoulder_pan_joint" value="1.54" />
-      <joint name="wrist_1_joint" value="-1.2" />
-      <joint name="wrist_2_joint" value="-1.6" />
-      <joint name="wrist_3_joint" value="-0.11" />
+      <joint name="${tf_prefix}elbow_joint" value="1.4" />
+      <joint name="${tf_prefix}shoulder_lift_joint" value="-1.62" />
+      <joint name="${tf_prefix}shoulder_pan_joint" value="1.54" />
+      <joint name="${tf_prefix}wrist_1_joint" value="-1.2" />
+      <joint name="${tf_prefix}wrist_2_joint" value="-1.6" />
+      <joint name="${tf_prefix}wrist_3_joint" value="-0.11" />
     </group_state>
     <!--END EFFECTOR - Purpose - Represent information about an end effector.-->
     <!--VIRTUAL JOINT - Purpose - this element defines a virtual joint between a robot link and an external frame of reference (considered fixed with respect to the robot)-->
     <!--DISABLE COLLISIONS - By default it is assumed that any link of the robot could potentially come into collision with any other link in the robot. This tag disables collision checking between a specified pair of links. -->
-    <disable_collisions link1="base_link" link2="base_link_inertia" reason="Adjacent" />
-    <disable_collisions link1="base_link_inertia" link2="shoulder_link" reason="Adjacent" />
-    <disable_collisions link1="tool0" link2="wrist_1_link" reason="Never" />
-    <disable_collisions link1="tool0" link2="wrist_2_link" reason="Never" />
-    <disable_collisions link1="tool0" link2="wrist_3_link" reason="Adjacent" />
-    <disable_collisions link1="forearm_link" link2="upper_arm_link" reason="Adjacent" />
-    <disable_collisions link1="forearm_link" link2="wrist_1_link" reason="Adjacent" />
-    <disable_collisions link1="shoulder_link" link2="upper_arm_link" reason="Adjacent" />
-    <disable_collisions link1="wrist_1_link" link2="wrist_2_link" reason="Adjacent" />
-    <disable_collisions link1="wrist_1_link" link2="wrist_3_link" reason="Never" />
-    <disable_collisions link1="wrist_2_link" link2="wrist_3_link" reason="Adjacent" />
+    <disable_collisions link1="${tf_prefix}base_link" link2="${tf_prefix}base_link_inertia" reason="Adjacent" />
+    <disable_collisions link1="${tf_prefix}base_link_inertia" link2="${tf_prefix}shoulder_link" reason="Adjacent" />
+    <disable_collisions link1="${tf_prefix}tool0" link2="${tf_prefix}wrist_1_link" reason="Never" />
+    <disable_collisions link1="${tf_prefix}tool0" link2="${tf_prefix}wrist_2_link" reason="Never" />
+    <disable_collisions link1="${tf_prefix}tool0" link2="${tf_prefix}wrist_3_link" reason="Adjacent" />
+    <disable_collisions link1="${tf_prefix}forearm_link" link2="${tf_prefix}upper_arm_link" reason="Adjacent" />
+    <disable_collisions link1="${tf_prefix}forearm_link" link2="${tf_prefix}wrist_1_link" reason="Adjacent" />
+    <disable_collisions link1="${tf_prefix}shoulder_link" link2="${tf_prefix}upper_arm_link" reason="Adjacent" />
+    <disable_collisions link1="${tf_prefix}wrist_1_link" link2="${tf_prefix}wrist_2_link" reason="Adjacent" />
+    <disable_collisions link1="${tf_prefix}wrist_1_link" link2="${tf_prefix}wrist_3_link" reason="Never" />
+    <disable_collisions link1="${tf_prefix}wrist_2_link" link2="${tf_prefix}wrist_3_link" reason="Adjacent" />
   </xacro:macro>
 </robot>
