Commit message: removed motion_primitive_ur.urdf.xacro and motion_primitive_ur_rsp.launch.py and added if else for driver_type to load the right ros2_control.xacro file in ur.urdf.xacro

File: ur_robot_driver/urdf/motion_primitive_ur.ros2_control.xacro (robot description, xacro)
@@ -4,5 +4,5 @@
   <xacro:include filename="$(find ur_robot_driver)/urdf/motion_primitive_ur_joint_control.xacro" />
   <xacro:include filename="$(find ur_description)/urdf/inc/ur_sensors.xacro" />
-  <xacro:macro name="motion_primitive_ur_ros2_control" params="
+  <xacro:macro name="ur_ros2_control" params="
     name
     tf_prefix

File: ur_robot_driver/urdf/ur.urdf.xacro (robot description, xacro)
@@ -3,7 +3,14 @@
   <!-- robot name parameter -->
   <xacro:arg name="name" default="ur"/>
+  <xacro:arg name="driver_type" default="standard" />
   <xacro:include filename="$(find ur_description)/urdf/ur_macro.xacro"/>
   <!-- ros2 control include -->
-  <xacro:include filename="$(find ur_robot_driver)/urdf/ur.ros2_control.xacro" />
+  <xacro:property name="driver_type" value="$(arg driver_type)" />
+  <xacro:if value="${driver_type == 'standard'}">
+    <xacro:include filename="$(find ur_robot_driver)/urdf/ur.ros2_control.xacro" />
+  </xacro:if>
+  <xacro:if value="${driver_type == 'motion_primitive'}">
+    <xacro:include filename="$(find ur_robot_driver)/urdf/motion_primitive_ur.ros2_control.xacro" />
+  </xacro:if>
   <xacro:include filename="$(find ur_description)/urdf/inc/ur_transmissions.xacro" />
   <!-- possible 'ur_type' values: ur3, ur3e, ur5, ur5e, ur10, ur10e, ur16e, ur20 -->
