Commit message: integrated motion_primitives_ur_driver into hardware_interface. build+launch succesfull. Executing primitives not working yet. Activating/ deactivating motion primitives mode during runtime not implemented yet.

File: ur_robot_driver/urdf/ur.ros2_control.xacro (robot description, xacro)
@@ -266,4 +266,33 @@
         <state_interface name="get_version_bugfix"/>
       </gpio>
+      <gpio name="motion_primitive">
+        <command_interface name="motion_type"/>
+        <command_interface name="q1"/>
+        <command_interface name="q2"/>
+        <command_interface name="q3"/>
+        <command_interface name="q4"/>
+        <command_interface name="q5"/>
+        <command_interface name="q6"/>
+        <command_interface name="pos_x"/>
+        <command_interface name="pos_y"/>
+        <command_interface name="pos_z"/>
+        <command_interface name="pos_qx"/>
+        <command_interface name="pos_qy"/>
+        <command_interface name="pos_qz"/>
+        <command_interface name="pos_qw"/>
+        <command_interface name="pos_via_x"/>
+        <command_interface name="pos_via_y"/>
+        <command_interface name="pos_via_z"/>
+        <command_interface name="pos_via_qx"/>
+        <command_interface name="pos_via_qy"/>
+        <command_interface name="pos_via_qz"/>
+        <command_interface name="pos_via_qw"/>
+        <command_interface name="blend_radius"/>
+        <command_interface name="velocity"/>
+        <command_interface name="acceleration"/>
+        <command_interface name="move_time"/>
+        <state_interface name="execution_status"/>
+        <state_interface name="ready_for_new_primitive"/>
+      </gpio>
     </ros2_control>
   </xacro:macro>

File: ur_robot_driver/urdf/ur.urdf.xacro (robot description, xacro)
@@ -3,16 +3,9 @@
   <!-- robot name parameter -->
   <xacro:arg name="name" default="ur"/>
-  <xacro:arg name="driver_type" default="standard" />
   <xacro:include filename="$(find ur_description)/urdf/ur_macro.xacro"/>
   <!-- ros2 control include -->
-  <xacro:property name="driver_type" value="$(arg driver_type)" />
-  <xacro:if value="${driver_type == 'standard'}">
-    <xacro:include filename="$(find ur_robot_driver)/urdf/ur.ros2_control.xacro" />
-  </xacro:if>
-  <xacro:if value="${driver_type == 'motion_primitive'}">
-    <xacro:include filename="$(find ur_robot_driver)/urdf/motion_primitive_ur.ros2_control.xacro" />
-  </xacro:if>
+  <xacro:include filename="$(find ur_robot_driver)/urdf/ur.ros2_control.xacro" />
   <xacro:include filename="$(find ur_description)/urdf/inc/ur_transmissions.xacro" />
-  <!-- possible 'ur_type' values: ur3, ur3e, ur5, ur5e, ur10, ur10e, ur16e, ur20 -->
+  <!-- possible 'ur_type' values: ur3, ur3e, ur5, ur5e, ur7e, ur10, ur10e, ur12e, ur16e, ur15, ur20, ur30 -->
   <!-- the default value should raise an error in case this was called without defining the type -->
   <xacro:arg name="ur_type" default="urXe"/>
