Commit message: Setup CM to not sleep and use blocking read

File: ur_robot_driver/urdf/ur.urdf.xacro (robot description, xacro)
@@ -31,4 +31,5 @@
   <xacro:arg name="script_sender_port" default="50002"/>
   <xacro:arg name="trajectory_port" default="50003"/>
+  <xacro:arg name="blocking_read" default="false" />
   <!--   tool communication related parameters-->
   <xacro:arg name="use_tool_communication" default="false" />
@@ -49,4 +50,5 @@
   <!-- convert to property to use substitution in function -->
   <xacro:property name="initial_positions_file" default="$(arg initial_positions_file)"/>
+  <xacro:property name="blocking_read" default="$(arg blocking_read)"/>
   <!-- create link fixed to the "world" -->
   <link name="world" />
@@ -93,4 +95,5 @@
     script_sender_port="$(arg script_sender_port)"
     trajectory_port="$(arg trajectory_port)"
+    non_blocking_read="${not blocking_read}"
   />
 </robot>
