Commit message: Use blocking read in controller manager (#1760)
* Setup CM to not sleep and use blocking read

* Change default value for blocking_read to true

* Updated documentation for blocking read functionality.

(cherry picked from commit c747f3ec6caee74f3bdc437ef93440a27299a404)

# Conflicts:
#	ur_robot_driver/doc/migration/makoa.rst
#	ur_robot_driver/urdf/ur.urdf.xacro

File: ur_robot_driver/urdf/ur.urdf.xacro (robot description, xacro)
@@ -31,5 +31,10 @@
   <xacro:arg name="script_sender_port" default="50002"/>
   <xacro:arg name="trajectory_port" default="50003"/>
+<<<<<<< HEAD
   <xacro:arg name="verify_robot_model" default="false" />
+=======
+  <xacro:arg name="verify_robot_model" default="true" />
+  <xacro:arg name="blocking_read" default="false" />
+>>>>>>> c747f3e (Use blocking read in controller manager (#1760))
   <!--   tool communication related parameters-->
   <xacro:arg name="use_tool_communication" default="false" />
@@ -50,4 +55,5 @@
   <!-- convert to property to use substitution in function -->
   <xacro:property name="initial_positions_file" default="$(arg initial_positions_file)"/>
+  <xacro:property name="blocking_read" default="$(arg blocking_read)"/>
   <!-- create link fixed to the "world" -->
   <link name="world" />
@@ -96,4 +102,5 @@
     ur_type="$(arg ur_type)"
     verify_robot_model="$(arg verify_robot_model)"
+    non_blocking_read="${not blocking_read}"
   />
 </robot>
